Commit message: URDF y STL modified

File: urdf/shadow_pa10_7dof.xacro (robot description, xacro)
@@ -171,6 +171,6 @@
 		<parent link="link_base"/>
 		<child link="link_s2"/>
-		<origin xyz="0 0 0.317" rpy="0 0 0" />
-		<axis xyz="0 0 -1" />
+		<origin xyz="0 0 0.317" rpy="0 0 3.14" />
+		<axis xyz="0 0 1" />
 		<limit effort="1000.0" lower="-3.09" upper="3.09" velocity="0.1"/>
 		<cfm>0.7</cfm>
@@ -912,5 +912,5 @@
 	    <parent link="inter"/>
 	    <child link="forearm"/>
-	    <origin xyz="0 0 0.055" rpy="0 0 1.57"/>
+	    <origin xyz="0 0 0.055" rpy="0 0 -1.57"/>
 	    <axis xyz="0 1 0"/>
 	    <!--<dynamics damping="0.7"/> -->
